File: schematics/benchBuddy.sch (KiCad schematic (older format))
At the start: 0 parts

Commit message: added fuses to power
Changed lines of the file:
@@
-EESchema Schematic File Version 2  date Sat 05 Oct 2013 10:55:51 PM EDT
+EESchema Schematic File Version 2  date Tue 08 Oct 2013 10:04:27 PM EDT
 LIBS:power
 LIBS:device
@@
 LIBS:contrib
 LIBS:valves
-LIBS:relays
 LIBS:benchBuddy-cache
 EELAYER 25  0
@@
 $Descr A4 11700 8267
 encoding utf-8
-Sheet 1 8
+Sheet 1 9
 Title ""
-Date "6 oct 2013"
+Date "9 oct 2013"
 Rev ""
 Comp ""
@@
 Comment4 ""
 $EndDescr
+$Sheet
+S 4800 850  1850 1200
+U 5254B562
+F0 "PowerAdjustmentMonitor" 60
+F1 "PowerAdjustmentMonitor.sch" 60
+$EndSheet
 $Sheet
 S 10300 1000 500  5800
@@
 $EndSheet
 $Sheet
-S 1650 1600 1850 1200
+S 650  650  1850 1200
 U 524F793A
 F0 "power" 60
